File: Rover_PCB.kicad_sch (KiCad schematic)
At the start: 138 parts, among them J1 XT90_24V_IN, J10 LED_RGY_B, J11 CAN_S1, J12 CAN_S2, J13 CAN_S3, J14 CAN_S4, J15 CAN_S5, J16 CAN_S6, J17 CAN7, J18 CAN8, J19 RJ45, J2 Brushed_Motor1, J20 Servo1, J21 Servo2, J22 Servo3, J23 Servo4, J24 Servo5, J25 Servo6, J26 Servo7, J27 Servo8, J28 UART1, J29 UART2, J3 Brushed_Motor2, J30 3.3V, J31 5V, J32 12V, J33 24V, J34 48V, J35 XT90_48V_IN, J36 Safety_Button, J37 STLINK, J38 USB_C_Receptacle_USB2.0_16P, J39 Load_Cell1, J4 LED_R_LL, J40 Load_Cell2, J41 Load_Cell3, J42 Load_Cell4, J43 XT90_24V_OUT, J44 XT90_48V_OUT, J45 ATX, J46 Conn_01x30_Socket, J47 FFC, J48 ATX, J49 Conn_01x30_Socket, J5 LED_R_LR, J50 FFC, J51 NTC1, J52 NTC2, J53 NTC3, J54 NTC4, J55 XT60_24V_OUT, J56 XT60_24V_OUT, J57 XT60_24V_OUT, J58 XT60_24V_OUT, J59 XT30_24V_OUT, J6 LED_R_RR, J60 XT30_24V_OUT, J61 XT30_24V_OUT, J62 XT30_24V_OUT, J63 XT60_48V_OUT, J64 XT60_48V_OUT, J65 XT60_12V_OUT, J66 XT60_12V_OUT, J67 XT30_48V_OUT, J68 XT30_48V_OUT, J69 XT30_12V_OUT, J7 LED_R_RL, J70 XT30_12V_OUT, J71 FFC, J72 FFC, J73 BAT1, J74 BAT_TOTAL, J8 LED_F_R, J9 LED_F_L, Q11 AO3400A, Q12 AO3400A, Q13 AO3400A, Q14 AO3400A, Q15 AO3400A, Q16 AO3400A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

Commit message: Aktualizacja schematu i PCB: dodanie rezonatora Y2, kondensatorow C9/C10 i punktow testowych J75-J79 oraz aktualizacja README.md i .gitignore
Parts:
- added C10, C9: 18pF, Capacitor_SMD:C_0603_1608Metric_Pad1.08x0.95mm_HandSolder, symbol Device:C
- added J75: TEST_PAD 5V, TestPoint:TestPoint_Pad_D1.5mm, symbol Connector:Conn_01x01_Pin
- added J76: TEST_PAD GND, TestPoint:TestPoint_Pad_D1.5mm, symbol Connector:Conn_01x01_Pin
- added J77: TEST_PAD 24V, TestPoint:TestPoint_Pad_D1.5mm, symbol Connector:Conn_01x01_Pin
- added J78: TEST_PAD 3.3V, TestPoint:TestPoint_Pad_D1.5mm, symbol Connector:Conn_01x01_Pin
- added J79: TEST_PAD 12V, TestPoint:TestPoint_Pad_D1.5mm, symbol Connector:Conn_01x01_Pin
- added Y2: 8MHz, Crystal:Crystal_SMD_3225-4Pin_3.2x2.5mm_HandSoldering, symbol Device:Crystal
Connections:
- net Pe12 is gone; now on net PE12: U12.11 (PD_SCK)
- net +12V: now also J79.1 (Pin_1)
- net +24V: now also J77.1 (Pin_1)
- net +3.3V: now also J78.1 (Pin_1)
- net +5V: now also J75.1 (Pin_1)
- net CANH_ETH: now also J19.1
- net CANL_ETH: now also J19.2
- net GND: now also C10.2, C9.2, J76.1 (Pin_1)
- net OUTA2: no longer J19.1
- net OUTB2: no longer J19.2
- net RX1: now also U1.25 (PA3)
- net RX2: now also U1.47 (PB11)
- net TX1: now also U1.24 (PA2)
- net TX2: now also U1.46 (PB10)
- net at U1.12 (PH0): now also C9.1, Y2.1
- net at U1.13 (PH1): now also C10.1, Y2.2
